File: eagle/stmboard.brd (EAGLE design)
At the start: 62.2 x 57.1 mm, 23 parts, among them IC1 LD117AS12TR

Commit message: some wiring touch-ups
Routing:
- net GND: track 13.7 -> 12.1 mm
Changed lines of the file:
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@@
 <wire x1="52.07" y1="5.08" x2="49.8475" y2="5.08" width="0.4572" layer="1"/>
 <via x="49.8475" y="5.08" extent="1-16" drill="0.75" diameter="1.524"/>
-<via x="48.133" y="-5.715" extent="1-16" drill="0.75" diameter="1.524"/>
+<via x="48.133" y="-4.1275" extent="1-16" drill="0.75" diameter="1.524"/>
 <contactref element="R3" pad="1"/>
 <contactref element="R4" pad="1"/>
@@
 <via x="70.485" y="-5.715" extent="1-16" drill="0.75" diameter="1.524"/>
 <wire x1="49.8475" y1="5.08" x2="48.133" y2="3.3655" width="0.4572" layer="16"/>
-<wire x1="48.133" y1="3.3655" x2="48.133" y2="-5.715" width="0.4572" layer="16"/>
+<wire x1="48.133" y1="3.3655" x2="48.133" y2="-4.1275" width="0.4572" layer="16"/>
 </signal>
 <signal name="PA4_AN">
@@
 <wire x1="43.18" y1="1.905" x2="42.545" y2="1.27" width="0.4572" layer="1"/>
 <wire x1="43.18" y1="11.85705625" x2="43.18" y2="1.905" width="0.4572" layer="1"/>
-<wire x1="23.495" y1="1.2065" x2="23.495" y2="1.27" width="0.4572" layer="1"/>
-<wire x1="23.495" y1="1.27" x2="23.495" y2="4.47" width="0.4572" layer="1"/>
-<wire x1="42.545" y1="1.27" x2="23.495" y2="1.27" width="0.4572" layer="1"/>
-<wire x1="23.241" y1="0.9525" x2="23.241" y2="-5.715" width="0.4572" layer="1"/>
-<wire x1="23.241" y1="0.9525" x2="23.495" y2="1.2065" width="0" layer="19" extent="1-1"/>
+<wire x1="42.545" y1="1.27" x2="24.765" y2="1.27" width="0.4572" layer="1"/>
+<wire x1="24.765" y1="1.27" x2="23.495" y2="2.54" width="0.4572" layer="1"/>
+<wire x1="23.495" y1="2.54" x2="23.495" y2="4.47" width="0.4572" layer="1"/>
+<wire x1="23.241" y1="-5.715" x2="23.241" y2="-0.254" width="0.4572" layer="1"/>
+<wire x1="23.241" y1="-0.254" x2="24.765" y2="1.27" width="0.4572" layer="1"/>
 </signal>
 <signal name="N$3">
