File: eagle/stmboard.brd (EAGLE design)
At the start: 62.2 x 57.1 mm, 23 parts, among them IC1 LD117AS12TR

Commit message: added part values
Parts:
- C1, C2: value (none) -> 27p
- C3: value (none) -> 10u
- C4: value (none) -> 10n
- C5, C6, C7: value (none) -> 100n
- IC1: value LD117AS12TR -> LD1117S33TR
- R2: value (none) -> 4K7
- R3: value (none) -> 82R
- R4: value (none) -> 68R
Changed lines of the file:
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@@
 </autorouter>
 <elements>
-<element name="C1" library="rcl" package="C1206" value="" x="69.85" y="32.385" smashed="yes" rot="R270">
+<element name="C1" library="rcl" package="C1206" value="27p" x="69.85" y="32.385" smashed="yes" rot="R270">
 <attribute name="NAME" x="71.12" y="33.655003125" size="1.27" layer="25" rot="R270"/>
 <attribute name="VALUE" x="67.309996875" y="33.655003125" size="1.27" layer="27" rot="R270"/>
 </element>
-<element name="C2" library="rcl" package="C1206" value="" x="69.85" y="26.035" smashed="yes" rot="R90">
+<element name="C2" library="rcl" package="C1206" value="27p" x="69.85" y="26.035" smashed="yes" rot="R90">
 <attribute name="NAME" x="68.58" y="24.764996875" size="1.27" layer="25" rot="R90"/>
 <attribute name="VALUE" x="72.390003125" y="24.764996875" size="1.27" layer="27" rot="R90"/>
 </element>
-<element name="C3" library="rcl" package="C1206K" value="" x="42.545" y="18.0975" smashed="yes" rot="R90">
+<element name="C3" library="rcl" package="C1206K" value="10u" x="42.545" y="18.0975" smashed="yes" rot="R90">
 <attribute name="NAME" x="41.445" y="16.4975" size="1.016" layer="25" rot="R90"/>
 <attribute name="VALUE" x="44.645" y="16.4975" size="1.016" layer="27" rot="R90"/>
 </element>
-<element name="C4" library="rcl" package="C1206K" value="" x="24.765" y="41.275" smashed="yes" rot="R180">
+<element name="C4" library="rcl" package="C1206K" value="10n" x="24.765" y="41.275" smashed="yes" rot="R180">
 <attribute name="NAME" x="28.27" y="38.905" size="1.016" layer="25" rot="R180"/>
 <attribute name="VALUE" x="26.365" y="43.375" size="1.016" layer="27" rot="R180"/>
 </element>
-<element name="C5" library="rcl" package="C1206K" value="" x="35.56" y="34.29" smashed="yes" rot="R180">
+<element name="C5" library="rcl" package="C1206K" value="100n" x="35.56" y="34.29" smashed="yes" rot="R180">
 <attribute name="NAME" x="37.16" y="35.73" size="1.016" layer="25" rot="R180"/>
 <attribute name="VALUE" x="37.16" y="36.39" size="1.016" layer="27" rot="R180"/>
 </element>
-<element name="C6" library="rcl" package="C1206K" value="" x="22.225" y="29.845" smashed="yes">
+<element name="C6" library="rcl" package="C1206K" value="100n" x="22.225" y="29.845" smashed="yes">
 <attribute name="NAME" x="20.625" y="30.945" size="1.016" layer="25"/>
 <attribute name="VALUE" x="20.625" y="27.745" size="1.016" layer="27"/>
 </element>
-<element name="IC1" library="v-reg" package="SOT223" value="LD117AS12TR" x="23.495" y="35.56" smashed="yes" rot="R90">
+<element name="IC1" library="v-reg" package="SOT223" value="LD1117S33TR" x="23.495" y="35.56" smashed="yes" rot="R90">
 <attribute name="NAME" x="23.4442" y="33.02" size="1.27" layer="25" rot="R90"/>
 <attribute name="VALUE" x="24.8158" y="33.02" size="1.27" layer="27" rot="R90"/>
 </element>
-<element name="R2" library="rcl" package="M1206" value="" x="69.85" y="8.89" smashed="yes" rot="R270">
+<element name="R2" library="rcl" package="M1206" value="4K7" x="69.85" y="8.89" smashed="yes" rot="R270">
 <attribute name="NAME" x="72.39" y="26.035" size="1.27" layer="25" rot="R270"/>
 <attribute name="VALUE" x="67.31" y="10.16" size="1.27" layer="27" rot="R270"/>
@@
 <attribute name="VALUE" x="69.469003125" y="23.494996875" size="1.27" layer="27" ratio="10" rot="R90"/>
 </element>
-<element name="C7" library="rcl" package="C1206K" value="" x="60.96" y="19.05" smashed="yes" rot="R270">
+<element name="C7" library="rcl" package="C1206K" value="100n" x="60.96" y="19.05" smashed="yes" rot="R270">
 <attribute name="NAME" x="62.06" y="20.650003125" size="1.016" layer="25" rot="R270"/>
 <attribute name="VALUE" x="58.86" y="20.65" size="1.016" layer="27" rot="R270"/>
@@
 <attribute name="VALUE" x="31.75" y="26.67" size="1.27" layer="27" rot="R180"/>
 </element>
-<element name="R3" library="rcl" package="M1206" value="" x="24.13" y="24.13" smashed="yes">
+<element name="R3" library="rcl" package="M1206" value="82R" x="24.13" y="24.13" smashed="yes">
 <attribute name="NAME" x="22.86" y="25.4" size="1.27" layer="25"/>
 <attribute name="VALUE" x="22.86" y="21.59" size="1.27" layer="27"/>
@@
 <attribute name="VALUE" x="26.67" y="18.415" size="1.27" layer="27" rot="R270"/>
 </element>
-<element name="R4" library="rcl" package="M1206" value="" x="29.21" y="11.43" smashed="yes" rot="R90">
+<element name="R4" library="rcl" package="M1206" value="68R" x="29.21" y="11.43" smashed="yes" rot="R90">
 <attribute name="NAME" x="27.94" y="10.16" size="1.27" layer="25" rot="R90"/>
 <attribute name="VALUE" x="31.75" y="10.16" size="1.27" layer="27" rot="R90"/>

Commit message: fixed SWDIO/SWCLK signal names
Connections:
- net PA13_SWCLK renamed PA13_SWDIO
- net PA14_SWDIO renamed PA14_SWCLK
Changed lines of the file:
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@@
 <wire x1="45.085" y1="31.75" x2="45.085" y2="28.2575" width="0.4572" layer="1"/>
 </signal>
-<signal name="PA14_SWDIO">
+<signal name="PA14_SWCLK">
 <contactref element="U$1" pad="24"/>
 <contactref element="JP8" pad="2"/>
@@
 <wire x1="55.88" y1="-2.54" x2="55.245" y2="-3.175" width="0.4572" layer="1"/>
 <wire x1="55.245" y1="-3.175" x2="55.245" y2="-5.715" width="0.4572" layer="1"/>
-</signal>
-<signal name="PA13_SWCLK">
-<contactref element="JP5" pad="7"/>
-<contactref element="U$1" pad="23"/>
-<contactref element="JP8" pad="4"/>
-<wire x1="50.448884375" y1="14.600459375" x2="48.26" y2="12.411575" width="0.4572" layer="1"/>
-<wire x1="48.26" y1="2.54" x2="52.07" y2="2.54" width="0.4572" layer="1"/>
-<wire x1="48.26" y1="12.411575" x2="48.26" y2="2.54" width="0.4572" layer="1"/>
-<wire x1="52.705" y1="-5.715" x2="52.705" y2="-4.1275" width="0.4572" layer="1"/>
-<wire x1="52.705" y1="-4.1275" x2="48.26" y2="0.3175" width="0.4572" layer="1"/>
-<wire x1="48.26" y1="2.54" x2="48.26" y2="0.3175" width="0.4572" layer="1"/>
 </signal>
 <signal name="PB5">
@@
 <wire x1="69.72" y1="10.16" x2="66.04" y2="10.16" width="0.4572" layer="1"/>
 </signal>
+<signal name="PA13_SWDIO">
+<contactref element="JP8" pad="4"/>
+<contactref element="U$1" pad="23"/>
+<contactref element="JP5" pad="7"/>
+<wire x1="50.448884375" y1="14.600459375" x2="48.26" y2="12.411575" width="0.4572" layer="1"/>
+<wire x1="48.26" y1="0.3175" x2="52.705" y2="-4.1275" width="0.4572" layer="1"/>
+<wire x1="52.705" y1="-4.1275" x2="52.705" y2="-5.715" width="0.4572" layer="1"/>
+<wire x1="48.26" y1="12.411575" x2="48.26" y2="2.54" width="0.4572" layer="1"/>
+<wire x1="48.26" y1="2.54" x2="48.26" y2="0.3175" width="0.4572" layer="1"/>
+<wire x1="52.07" y1="2.54" x2="48.26" y2="2.54" width="0.4572" layer="1"/>
+</signal>
 </signals>

Commit message: fixed value labels on brd
Parts:
- C4: value 10n -> 100n
Changed lines of the file:
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@@
 <layer number="25" name="tNames" color="7" fill="1" visible="no" active="yes"/>
 <layer number="26" name="bNames" color="7" fill="1" visible="no" active="yes"/>
-<layer number="27" name="tValues" color="7" fill="1" visible="no" active="yes"/>
+<layer number="27" name="tValues" color="7" fill="1" visible="yes" active="yes"/>
 <layer number="28" name="bValues" color="7" fill="1" visible="no" active="yes"/>
 <layer number="29" name="tStop" color="7" fill="3" visible="no" active="yes"/>
@@
 <element name="C1" library="rcl" package="C1206" value="27p" x="69.85" y="32.385" smashed="yes" rot="R270">
 <attribute name="NAME" x="71.12" y="33.655003125" size="1.27" layer="25" rot="R270"/>
-<attribute name="VALUE" x="67.309996875" y="33.655003125" size="1.27" layer="27" rot="R270"/>
+<attribute name="VALUE" x="71.754996875" y="33.655003125" size="1.27" layer="27" rot="R270"/>
 </element>
 <element name="C2" library="rcl" package="C1206" value="27p" x="69.85" y="26.035" smashed="yes" rot="R90">
 <attribute name="NAME" x="68.58" y="24.764996875" size="1.27" layer="25" rot="R90"/>
-<attribute name="VALUE" x="72.390003125" y="24.764996875" size="1.27" layer="27" rot="R90"/>
+<attribute name="VALUE" x="73.025003125" y="24.764996875" size="1.27" layer="27" rot="R90"/>
 </element>
 <element name="C3" library="rcl" package="C1206K" value="10u" x="42.545" y="18.0975" smashed="yes" rot="R90">
 <attribute name="NAME" x="41.445" y="16.4975" size="1.016" layer="25" rot="R90"/>
-<attribute name="VALUE" x="44.645" y="16.4975" size="1.016" layer="27" rot="R90"/>
-</element>
-<element name="C4" library="rcl" package="C1206K" value="10n" x="24.765" y="41.275" smashed="yes" rot="R180">
+<attribute name="VALUE" x="25.3875" y="28.38" size="1.016" layer="27"/>
+</element>
+<element name="C4" library="rcl" package="C1206K" value="100n" x="24.765" y="41.275" smashed="yes" rot="R180">
 <attribute name="NAME" x="28.27" y="38.905" size="1.016" layer="25" rot="R180"/>
-<attribute name="VALUE" x="26.365" y="43.375" size="1.016" layer="27" rot="R180"/>
+<attribute name="VALUE" x="25.095" y="44.01" size="1.016" layer="27" rot="R180"/>
 </element>
 <element name="C5" library="rcl" package="C1206K" value="100n" x="35.56" y="34.29" smashed="yes" rot="R180">
 <attribute name="NAME" x="37.16" y="35.73" size="1.016" layer="25" rot="R180"/>
-<attribute name="VALUE" x="37.16" y="36.39" size="1.016" layer="27" rot="R180"/>
+<attribute name="VALUE" x="35.89" y="37.025" size="1.016" layer="27" rot="R180"/>
 </element>
 <element name="C6" library="rcl" package="C1206K" value="100n" x="22.225" y="29.845" smashed="yes">
 <attribute name="NAME" x="20.625" y="30.945" size="1.016" layer="25"/>
-<attribute name="VALUE" x="20.625" y="27.745" size="1.016" layer="27"/>
+<attribute name="VALUE" x="40.835" y="16.815" size="1.016" layer="27" rot="R90"/>
 </element>
 <element name="IC1" library="v-reg" package="SOT223" value="LD1117S33TR" x="23.495" y="35.56" smashed="yes" rot="R90">
 <attribute name="NAME" x="23.4442" y="33.02" size="1.27" layer="25" rot="R90"/>
-<attribute name="VALUE" x="24.8158" y="33.02" size="1.27" layer="27" rot="R90"/>
+<attribute name="VALUE" x="18.4658" y="29.845" size="1.27" layer="27" rot="R90"/>
 </element>
 <element name="R2" library="rcl" package="M1206" value="4K7" x="69.85" y="8.89" smashed="yes" rot="R270">
 <attribute name="NAME" x="72.39" y="26.035" size="1.27" layer="25" rot="R270"/>
-<attribute name="VALUE" x="67.31" y="10.16" size="1.27" layer="27" rot="R270"/>
+<attribute name="VALUE" x="71.755" y="10.16" size="1.27" layer="27" rot="R270"/>
 </element>
 <element name="U$1" library="stm32F030x" package="TQFP32-08" package3d_urn="urn:adsk.eagle:package:4313/2" value="STM32F030" x="52.07" y="19.05" smashed="yes" rot="R225">
 <attribute name="NAME" x="57.619803125" y="17.415590625" size="0.8128" layer="25" rot="R225"/>
-<attribute name="VALUE" x="53.309278125" y="22.085321875" size="0.8128" layer="27" rot="R225"/>
+<attribute name="VALUE" x="52.674278125" y="22.720321875" size="0.8128" layer="27" rot="R225"/>
 </element>
 <element name="Q2" library="crystal" package="SM49" value="" x="65.405" y="29.21" smashed="yes" rot="R90">
@@
 <element name="C7" library="rcl" package="C1206K" value="100n" x="60.96" y="19.05" smashed="yes" rot="R270">
 <attribute name="NAME" x="62.06" y="20.650003125" size="1.016" layer="25" rot="R270"/>
-<attribute name="VALUE" x="58.86" y="20.65" size="1.016" layer="27" rot="R270"/>
+<attribute name="VALUE" x="62.67" y="19.38" size="1.016" layer="27" rot="R270"/>
 </element>
 <element name="S2" library="SparkFun-Switches" package="TACTILE_SWITCH_SMD_6.0X3.5MM" value="" x="33.655" y="29.845" smashed="yes">
@@
 <element name="R3" library="rcl" package="M1206" value="82R" x="24.13" y="24.13" smashed="yes">
 <attribute name="NAME" x="22.86" y="25.4" size="1.27" layer="25"/>
-<attribute name="VALUE" x="22.86" y="21.59" size="1.27" layer="27"/>
+<attribute name="VALUE" x="22.225" y="21.59" size="1.27" layer="27"/>
 </element>
 <element name="LED2" library="led" library_urn="urn:adsk.eagle:library:259" package="1206" package3d_urn="urn:adsk.eagle:package:15796/2" value="" x="29.21" y="17.145" smashed="yes" rot="R270">
@@
 <element name="R4" library="rcl" package="M1206" value="68R" x="29.21" y="11.43" smashed="yes" rot="R90">
 <attribute name="NAME" x="27.94" y="10.16" size="1.27" layer="25" rot="R90"/>
-<attribute name="VALUE" x="31.75" y="10.16" size="1.27" layer="27" rot="R90"/>
+<attribute name="VALUE" x="27.305" y="10.795" size="1.27" layer="27" rot="R90"/>
 </element>
 <element name="S1" library="SparkFun-Switches" package="TACTILE_SWITCH_SMD_6.0X3.5MM" value="" x="23.495" y="7.62" smashed="yes" rot="R270">
